File: RCM-CommX1/RCM-CommV2.brd (EAGLE design)
At the start: 50.8 x 66 mm, 25 parts, among them J1 BLACKFIN_HEADER, J2- C-GRID-04

Commit message: Version 2.0 of RCM-Comm board ready for review.
Parts:
- removed C3: 1000pF, spark_fun:0603-CAP
- removed FX1: S558-5999-T7-F, halo-electronics:N5
- removed J2-: C-GRID-04, MolexConnector:70555-04
- removed LED_3V3_, LED_ENET_ACT_, LED_ENET_LINK_, LED_WLAN_STATUS_: (no value), spark_fun:LED-0603
- removed U$1: LANTRONIX_XPICO, xPico:LANTRONIX_XPICO
- added C1, C4, C5, C8, C9: 0.1uF, SparkFun-Capacitors:0603-CAP
- added C6, C7: 10uF, SparkFun-Capacitors:0603-CAP
- added J3: USB-MICROB, SparkFun-Connectors:USB-MICROB
- added J4: (no value), SparkFun-Connectors:1X02_LOCK
- added J5, J6: (no value), SparkFun-Connectors:1X06_LOCK
- added JP3, JP4, JP5, JP6: JUMPER-PAD-2-NOROUND, SparkFun-Passives:PAD-JUMPER-2-NO_YES_SILK_ROUND
- added LED1, LED2, LED3: GREEN, spark_fun:LED-0603
- added S1: WAKE, SparkFun-Electromechanical:TACTILE-SWITCH-SMD
- added S2: DEFAULTS, SparkFun-Electromechanical:TACTILE-SWITCH-SMD
- added S3: RESET, SparkFun-Electromechanical:TACTILE-SWITCH-SMD
- added U1: LANTRONIX_XPICO, xPico:LANTRONIX_XPICO
- C2: device rcl:C0603 -> SparkFun-Capacitors:0603-CAP
- R4: value 330 -> 1K; device spark_fun:0603-RES -> rcl:R0603
- moved U$3 63.2 mm to (19.4, 29.6)
- moved LOGO1 51.1 mm to (17.8, 38.1)
- moved R3 49.0 mm to (21.6, 58.4)
- moved C2 44.9 mm to (12.7, 31.1), turned to 0 degrees
- moved R5 44.0 mm to (31.8, 58.4)
- moved R6 37.0 mm to (26.7, 58.4)
- moved JP1 27.9 mm to (16.5, 10.2), turned to 180 degrees
- moved R1 26.4 mm to (12.7, 10.2)
- moved JP2 21.7 mm to (16.5, 15.2), turned to 0 degrees
- moved R2 20.1 mm to (12.7, 15.2)
- moved R4 19.1 mm to (12.7, 34.9), turned to 180 degrees
- moved FID1 1.27 mm to (5.08, 3.81)
- moved FID3 1.27 mm to (50.8, 3.81)
Connections:
- removed net ACT: R5.1, U$1.P8
- removed net ERCT: FX1.10, U$1.P18
- removed net ETCT: FX1.15, U$1.P12
- removed net LINK: R4.1
- removed net N$13: FX1.16, U$1.P13
- removed net N$14: FX1.14, U$1.P11
- removed net N$16: FX1.11, U$1.P19
- removed net N$17: FX1.9, U$1.P17
- removed net N$18: FX1.1, J2-.4
- removed net N$19: FX1.3, J2-.3
- removed net N$20: FX1.8, J2-.1
- removed net N$21: FX1.6, J2-.2
- removed net N$7: U$1.P6
- removed net WLAN: R6.1, U$1.P4
- new net !DEFAULT!: C2.1, S2.3, U1.P36
- new net !EXT_RESET!: C8.1, S3.3, U1.P38
- new net BF_CLK: J1.11, JP4.1
- new net BF_CS: J1.12, JP6.2
- new net BF_MISO: J1.10, JP5.2
- new net BF_MOSI: J1.9, JP3.1
- new net CP1: J6.1, U1.P35
- new net CP2/SPI_INT: J6.2, U1.P26
- new net CP3/MISO: J6.3, JP3.2, U1.P28
- new net CP4/MOSI: J6.4, JP5.1, U1.P30
- new net CP5: J5.1, U1.P32
- new net CP6: J5.2, U1.P34
- new net CP7/SPI_SCK: J5.3, JP4.2, U1.P27
- new net CP8/SPI_CS: J5.4, JP6.1, U1.P3
- new net DDM: J3.D-, U1.P24
- new net DDP: J3.D+, U1.P22
- new net SYSTEM_LED: R5.1, U1.P20
- new net WKUP: C9.1, S1.3, U1.P14
- new net WLAN_LED: R6.1, U1.P4
- net CTS1: now also U1.P16; no longer U$1.P16
- net GND: now also C1.2, C4.2, C5.2, C6.2, C7.2, C8.2, C9.2, J3.GND, J3.MT1, J3.MT2, J4.1, J5.6, J6.6, LED2.C, S3.1, U1.P1, U1.P15, U1.P2, U1.P21, U1.P37, U1.P39, U1.P40, U1.P9; no longer C3.2, U$1.P1, U$1.P15, U$1.P2, U$1.P21, U$1.P37, U$1.P39, U$1.P40, U$1.P9
- net N$1: now also J4.2, S2.1; no longer C3.1, FX1.2, FX1.7
- net N$3: now also LED1.C; no longer LED_3V3_.C
- net N$5: now also S1.1; no longer LED_ENET_LINK_.C
- net N$6: now also LED2.A; no longer LED_ENET_ACT_.C
- net N$8: now also LED3.C; no longer LED_WLAN_STATUS_.C
- net RTS1: now also U1.P5; no longer U$1.P5
- net RXD1: now also U1.P7; no longer U$1.P7
- net RXD2: now also U1.P23; no longer U$1.P23
- net TXD1: now also U1.P10; no longer U$1.P10
- net TXD2: now also U1.P25; no longer U$1.P25
- net VCC: now also C1.1, C4.1, C5.1, C6.1, C7.1, J5.5, J6.5, LED1.A, LED3.A, R4.1, U1.P29, U1.P31, U1.P33; no longer C2.1, LED_3V3_.A, LED_ENET_ACT_.A, LED_ENET_LINK_.A, LED_WLAN_STATUS_.A, U$1.P29, U$1.P31, U$1.P33
Routing:
- net BF_CS: track 0.00 -> 58.4 mm, vias 0 -> 2
- net BF_MISO: track 0.00 -> 58.0 mm, vias 0 -> 2
- net CP4/MOSI: track 0.00 -> 57.4 mm, vias 0 -> 2
- net CP7/SPI_SCK: track 0.00 -> 53.6 mm, vias 0 -> 3
- net CP3/MISO: track 0.00 -> 53.3 mm, vias 0 -> 2
- net BF_CLK: track 0.00 -> 51.4 mm, vias 0 -> 2
- net BF_MOSI: track 0.00 -> 50.9 mm, vias 0 -> 2
- net CP1: track 0.00 -> 49.4 mm, vias 0 -> 1
- net CP2/SPI_INT: track 0.00 -> 49.0 mm, vias 0 -> 1
- net !DEFAULT!: track 0.00 -> 43.0 mm, vias 0 -> 2
- net SYSTEM_LED: track 0.00 -> 40.6 mm, vias 0 -> 2
- net WLAN_LED: track 0.00 -> 39.5 mm, vias 0 -> 2
- net CP6: track 0.00 -> 38.9 mm, vias 0 -> 1
- net WKUP: track 0.00 -> 38.8 mm, vias 0 -> 2
- net VCC: track 0.00 -> 37.5 mm, vias 0 -> 5
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Other:
- board text added: "CP1"
- board text added: "CP2"
- board text added: "CP3"
- board text added: "CP4"
- board text added: "CP5"
- board text added: "CP6"
- board text added: "CP7"
- board text added: "CP8"
- board text added: "DEAFAULT"
- board text added: "E^3 RCM-Comm v2.0 (c) 2016"
- board text added: "Engineering^3, 2016 http://engineering3.org"
- board text added: "GND"
- board text added: "MISO"
- board text added: "MOSI"
- board text added: "RESET"
- board text added: "RXD2"
- board text added: "RoHS Compliant"
- board text added: "SPI_CS"
- board text added: "SPI_SCK"
- board text added: "SYS"
- board text added: "TXD2"
- board text added: "WAKE"
- board text removed: "ACT"
- board text removed: "Copyright 2015 Engineering^3"
- board text removed: "LINK"
- board text removed: "RCM-Comm v1 (c) 2014, 2015"
