File: RCM-Comm_v2/RCM-CommV2.sch (EAGLE design)
At the start: 39 parts, among them J1 BLACKFIN_HEADER, J3 USB-MICROB, U1 LANTRONIX_XPICO

Commit message: Fixed attribution text in schematic.
Other:
- note added: "Designed for Tim Jump of Engineering^3 by Brian Schmalz of Schmalz Haus LLC"
- note removed: "Designed for Tim Jump of Engineering^3 by Brian Schmalz of Logic PD"
Changed lines of the file:
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@@
 <plain>
 <text x="150.368" y="29.21" size="1.778" layer="98">Designed for Tim Jump of Engineering^3
-by Brian Schmalz of Logic PD</text>
+by Brian Schmalz of Schmalz Haus LLC</text>
 <text x="149.86" y="25.4" size="1.778" layer="98">Copyright 2016 Engineering^3 LLC</text>
 <text x="5.08" y="162.56" size="1.27" layer="98">Copyright 2016 Engineering^3 LLC Copyright and related rights are licensed under the Solderpad Hardware License,
